File: MFOS_ADSR/MFOS_ADSR.kicad_sch (KiCad schematic)
At the start: 68 parts, among them J1 AudioJack2, J10 Conn_01x01, J11 Conn_01x01, J12 Conn_01x01, J13 Conn_01x01, J14 Conn_01x01, J15 Conn_01x01, J2 AudioJack2, J3 AudioJack2, J4 Conn_01x01, J5 Conn_01x01, J6 Conn_01x01, J7 Conn_01x01, J8 Conn_01x01, J9 Conn_01x01, U1 TL082, U2 4001, U3 40106, U4 4066, U5 TL084

Commit message: Revision until and with audio mixer complete
Parts:
- removed J1, J2, J3: AudioJack2, symbol Connector:AudioJack2
- removed S1: SW_SPST, symbol Switch:SW_SPST
- added J1, J2, J3: Jack-DC, symbol Connector:Jack-DC
- added S1: SW_Push, symbol Switch:SW_Push
- J10, J11, J12, J13, J14, J15, J4, J5, J6, J7, J8, J9: now left out of the parts list
Connections:
- net GAT: now also J2.2
- net GND: now also J1.1, J2.1, J3.1, S1.2
- net MGT: now also S1.1
- net TRG: now also J1.2
- net at R24.1: now also J3.2
