File: MFOS_VCA/MFOS_VCA.kicad_sch (KiCad schematic)
At the start: 88 parts, among them J1 Jack-DC, J10 Conn_01x01, J11 Conn_01x01, J12 Conn_01x01, J13 Conn_01x01, J14 Conn_01x01, J15 Conn_01x01, J16 Conn_01x01, J17 Conn_01x01, J18 Conn_01x01, J19 Conn_01x01, J2 Jack-DC, J20 Conn_01x01, J21 Conn_01x01, J22 Conn_01x01, J23 Conn_01x01, J24 Conn_01x01, J3 Conn_01x01, J4 Jack-DC, J5 Jack-DC, J6 Jack-DC, J7 Conn_01x01, J8 Jack-DC, J9 Conn_01x01, Q1 2N3904, Q2 2N3906, Q3 2N3904, Q4 2N3906, SW1 SW_SPDT, SW2 SW_SPDT, U1 TL084, U2 LM13700

Commit message: Reviewed BOM
Parts:
- J10, J11, J12, J13, J14, J15, J16, J17, J18, J19, J20, J21, J22, J23, J24, J3, J7, J9: now left out of the parts list
- R18, R41, R45, R47: symbol Device:R_Potentiometer -> dhk:R_Potentiometer_Trim
