File: MFOS_VCO/untitled.kicad_sch (KiCad schematic)
At the start: 0 parts

Commit message: Final changes
Parts:
- added C1, C15, C16, C2: 0.1uF, symbol Device:C
- added C12, C13: 1uF, symbol dhk:C_Tantalum
- added C14: 0.002uF, symbol Device:C
- added C4: 10pF, symbol Device:C
- added D2, D3, D4, D5, D6, D7: 1N914, Diode_THT:D_DO-35_SOD27_P7.62mm_Horizontal, symbol Diode:1N914
- added R1, R12, R13, R25, R32, R35, R40: 10k, symbol Device:R
- added R14, R21, R48: 20k, symbol Device:R
- added R20: 47k, symbol Device:R
- added R22, R26, R49, R51: 1k, symbol Device:R
- added R29, R44, R6, R67: 100k, symbol Device:R
- added R36, R52: 4.7k, symbol Device:R
- added R39: 100k, symbol Device:R_Potentiometer
- added R41: 3k, symbol Device:R
- added R45: 1M, symbol Device:R
- added R5, R7: 10k, symbol dhk:R_Potentiometer_Trim_Top
- added R53: 130k, symbol Device:R
- added R59: 1M, symbol dhk:R_Potentiometer_Trim_Top
- added R60, R64: 100k, symbol dhk:R_Potentiometer_Trim_Top
- added R61: 470k, symbol Device:R
- added R68: 10M, symbol Device:R
- added U4: TL074, symbol Amplifier_Operational:TL074
- added U5: LM13700, symbol Amplifier_Operational:LM13700
- added U6: TL072, symbol Amplifier_Operational:TL072
- added U7: TL071, symbol Amplifier_Operational:TL071
Connections:
- new net: C14.1, D2.1 (K), D3.1 (K), R13.1, R21.1
- new net: D3.2 (A), D4.2 (A), D7.1 (K), R26.1, R29.1, R32.2, U4.7
- new net: C4.2, R36.1, R68.2, U7.6
- new net: R45.2, R53.1, U5.5, U5.7
- new net: R25.1, R32.1, U4.6 (-)
- new net: D2.2 (A), R20.2, R25.2, U4.1
- new net: D5.1 (K), D6.2 (A)
- new net: C12.2, D5.2 (A), U6.5 (+)
- new net: D6.1 (K), D7.2 (A)
- new net: R60.2, R61.1
- new net: C1.1, R5.2, U4.3 (+)
- new net: R35.1, R40.2, U7.2 (-)
- new net: R35.2, R39.2
- new net: R49.1, R52.1, U5.8
- new net: R48.2, R51.1, R61.2, U5.3 (+)
- new net: C2.1, R7.2, U4.10 (+)
- new net: R14.2, R22.1, R64.3, U4.8
- new net: R13.2, R14.1, U4.9 (-)
- new net: R39.1, U6.6 (-), U6.7
- new net: R39.3, U6.1, U6.2 (-)
- new net: R1.1, R7.3
- new net: R5.3, R6.1
- new net: C13.1, D4.1 (K), U6.3 (+)
- new net: C4.1, R29.2, R68.1, U7.3 (+)
- new net: U4.13 (-), U4.14
- new net: R44.1, R59.1, R59.2
- new net: R48.1, R64.1, R64.2
- new net: R12.2, R20.1, U4.2 (-)
- new net: R44.2, U5.1
- new net +12V: C15.1, R1.2, R45.1, R59.3, R6.2, R60.3, U7.7 (V+)
- new net -12V: C14.2, C16.1, R21.2, R52.2, R60.1, U7.4 (V-)
- new net GND: C1.2, C12.1, C13.2, C15.2, C16.2, C2.2, R41.2, R5.1, R51.2, R53.2, R67.1, R7.1, U4.12 (+), U4.5 (+), U5.13 (-), U5.14 (+), U5.4 (-)
- new net PWM: R40.1, R67.2
- new net RAW: R12.1
- new net RMP: R26.2
- new net SIN: R49.2
- new net SQR: R36.2, R41.1
- new net TRI: R22.2
- no-connect marks 0 -> 8

Commit message: Lots of headway
Parts:
- added J27: Conn_01x03, Connector_PinHeader_2.54mm:PinHeader_1x03_P2.54mm_Vertical, symbol Connector_Generic:Conn_01x03
- C1, C15, C16, C2: footprint (none) -> Capacitor_THT:C_Disc_D5.0mm_W2.5mm_P2.50mm
- C12, C13: footprint (none) -> Capacitor_THT:CP_Radial_D8.0mm_P3.50mm
- C14: footprint (none) -> Capacitor_THT:C_Disc_D4.7mm_W2.5mm_P5.00mm
- C4: footprint (none) -> Capacitor_THT:C_Disc_D3.4mm_W2.1mm_P2.50mm
- R1, R12, R13, R14, R20, R21, R22, R25, R26, R29, R32, R35, R36, R39, R40, R41, R44, R45, R48, R49, R51, R52, R53, R6, R61, R67, R68, R7: footprint (none) -> Resistor_THT:R_Axial_DIN0207_L6.3mm_D2.5mm_P7.62mm_Horizontal
- R5, R59, R60, R64: footprint (none) -> Potentiometer_THT:Potentiometer_Bourns_3339P_Vertical
- U4: footprint (none) -> Package_DIP:DIP-14_W7.62mm_Socket_LongPads
- U5: footprint (none) -> Package_SO:SOIC-16_3.9x9.9mm_P1.27mm
- U6, U7: footprint (none) -> Package_DIP:DIP-8_W7.62mm_Socket_LongPads
Connections:
- net R39P2: now reaches R35.2, R39.2
- net R39P2: now also J27.2 (Pin_2)
- net R39P1: now reaches R39.1, U6.6 (-), U6.7
- net R39P1: now also J27.1 (Pin_1)
- net R39P3: now reaches R39.3, U6.1, U6.2 (-)
- net R39P3: now also J27.3 (Pin_3)

Commit message: Laying out
Parts:
- R7: footprint Resistor_THT:R_Axial_DIN0207_L6.3mm_D2.5mm_P7.62mm_Horizontal -> Potentiometer_THT:Potentiometer_Bourns_3339P_Vertical
Changed lines of the file:
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@@
     (property "Reference" "R7" (id 0) (at 99.06 50.8 90))
     (property "Value" "10k" (id 1) (at 99.06 53.34 90))
-    (property "Footprint" "Resistor_THT:R_Axial_DIN0207_L6.3mm_D2.5mm_P7.62mm_Horizontal" (id 2) (at 99.06 57.15 0)
+    (property "Footprint" "Potentiometer_THT:Potentiometer_Bourns_3339P_Vertical" (id 2) (at 99.06 57.15 0)
       (effects (font (size 1.27 1.27)) hide)
     )
