File: MFOS_VCO/untitled.kicad_sch (KiCad schematic)
At the start: 51 parts, among them J27 Conn_01x03, U4 TL074, U5 LM13700, U6 TL072, U7 TL071

Commit message: Fixed PN4391 bug. Made some layout changes. Fitted molex connectors instead of pin connectors
Parts:
- C12: footprint Capacitor_THT:CP_Radial_D8.0mm_P3.50mm -> Capacitor_THT:CP_Radial_D5.0mm_P2.00mm
- C13: footprint Capacitor_THT:CP_Radial_D8.0mm_P3.50mm -> Capacitor_THT:CP_Radial_D5.0mm_P2.50mm
Changed lines of the file:
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@@
     (property "Reference" "C13" (id 0) (at 160.02 97.79 90))
     (property "Value" "1uF" (id 1) (at 165.1 97.79 90))
-    (property "Footprint" "Capacitor_THT:CP_Radial_D8.0mm_P3.50mm" (id 2) (at 165.1 100.6348 0)
+    (property "Footprint" "Capacitor_THT:CP_Radial_D5.0mm_P2.50mm" (id 2) (at 165.1 100.6348 0)
       (effects (font (size 1.27 1.27)) hide)
     )
@@
     (property "Reference" "C12" (id 0) (at 160.02 110.49 90))
     (property "Value" "1uF" (id 1) (at 165.1 110.49 90))
-    (property "Footprint" "Capacitor_THT:CP_Radial_D8.0mm_P3.50mm" (id 2) (at 157.48 107.6452 0)
-      (effects (font (size 1.27 1.27)) hide)
-    )
+    (property "Footprint" "Capacitor_THT:CP_Radial_D5.0mm_P2.00mm" (id 2) (at 157.48 107.6452 0)
+      (effects (font (size 1.27 1.27)) hide)
+    )

Commit message: Some bugfixes
Parts:
- J27: footprint Connector_PinHeader_2.54mm:PinHeader_1x03_P2.54mm_Vertical -> Connector_Molex:Molex_KK-254_AE-6410-03A_1x03_P2.54mm_Vertical
Changed lines of the file:
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@@
       (effects (font (size 1.27 1.27)) (justify left) hide)
     )
-    (property "Footprint" "Connector_PinHeader_2.54mm:PinHeader_1x03_P2.54mm_Vertical" (id 2) (at 238.76 118.11 0)
+    (property "Footprint" "Connector_Molex:Molex_KK-254_AE-6410-03A_1x03_P2.54mm_Vertical" (id 2) (at 238.76 118.11 0)
       (effects (font (size 1.27 1.27)) hide)
     )
